Commit message: foot friction changed

File: robots/a1_description/xacro/const.xacro (robot description, xacro)
@@ -90,3 +90,9 @@
     <!-- foot -->
     <xacro:property name="foot_mass" value="0.06"/>
+    <!-- foot friction -->
+    <xacro:property name="foot_mu1" value="1.0"/>
+    <xacro:property name="foot_mu2" value="1.0"/>
+    <xacro:property name="foot_minDepth" value="0.0002"/>
+    <xacro:property name="foot_kp" value="1000000.0"/>
+    <xacro:property name="foot_kd" value="100.0"/>
 </robot>

File: robots/a1_description/xacro/gazebo.xacro (robot description, xacro)
@@ -161,10 +161,10 @@
     </gazebo>
     <gazebo reference="FL_foot">
-        <mu1>0.6</mu1>
-        <mu2>0.6</mu2>
-        <self_collide>1</self_collide>
-        <material>Gazebo/DarkGrey</material>
-        <kp  value="1000000.0"/>
-        <kd  value="1.0"/>
+        <mu1>${foot_mu1}</mu1>
+        <mu2>${foot_mu2}</mu2>
+        <self_collide>1</self_collide>
+        <material>Gazebo/DarkGrey</material>
+        <kp  value="${foot_kp}"/>
+        <kd  value="${foot_kd}"/>
     </gazebo>
     <!-- FR leg -->
@@ -188,10 +188,10 @@
     </gazebo>
     <gazebo reference="FR_foot">
-        <mu1>0.6</mu1>
-        <mu2>0.6</mu2>
-        <self_collide>1</self_collide>
-        <material>Gazebo/DarkGrey</material>
-        <kp  value="1000000.0"/>
-        <kd  value="1.0"/>
+        <mu1>${foot_mu1}</mu1>
+        <mu2>${foot_mu2}</mu2>
+        <self_collide>1</self_collide>
+        <material>Gazebo/DarkGrey</material>
+        <kp  value="${foot_kp}"/>
+        <kd  value="${foot_kd}"/>
     </gazebo>
     <!-- RL leg -->
@@ -215,10 +215,10 @@
     </gazebo>
     <gazebo reference="RL_foot">
-        <mu1>0.6</mu1>
-        <mu2>0.6</mu2>
-        <self_collide>1</self_collide>
-        <material>Gazebo/DarkGrey</material>
-        <kp  value="1000000.0"/>
-        <kd  value="1.0"/>
+        <mu1>${foot_mu1}</mu1>
+        <mu2>${foot_mu2}</mu2>
+        <self_collide>1</self_collide>
+        <material>Gazebo/DarkGrey</material>
+        <kp  value="${foot_kp}"/>
+        <kd  value="${foot_kd}"/>
     </gazebo>
     <!-- RR leg -->
@@ -242,10 +242,10 @@
     </gazebo>
     <gazebo reference="RR_foot">
-        <mu1>0.6</mu1>
-        <mu2>0.6</mu2>
-        <self_collide>1</self_collide>
-        <material>Gazebo/DarkGrey</material>
-        <kp  value="1000000.0"/>
-        <kd  value="1.0"/>
+        <mu1>${foot_mu1}</mu1>
+        <mu2>${foot_mu2}</mu2>
+        <self_collide>1</self_collide>
+        <material>Gazebo/DarkGrey</material>
+        <kp  value="${foot_kp}"/>
+        <kd  value="${foot_kd}"/>
     </gazebo>
 </robot>

Commit message: urdf same as pybullet

File: robots/a1_description/xacro/const.xacro (robot description, xacro)
@@ -24,5 +24,5 @@
     <xacro:property name="calf_length" value="0.2"/>
     <!-- leg offset from trunk center value -->
-    <xacro:property name="leg_offset_x" value="0.1805"/>
+    <xacro:property name="leg_offset_x" value="0.183"/>
     <xacro:property name="leg_offset_y" value="0.047"/>
     <xacro:property name="trunk_offset_z" value="0.01675"/>
@@ -33,14 +33,14 @@
     <xacro:property name="hip_max" value="46"/>
     <xacro:property name="hip_min" value="-46"/>
-    <xacro:property name="hip_velocity_max" value="21"/>
-    <xacro:property name="hip_torque_max" value="33.5"/>
+    <xacro:property name="hip_velocity_max" value="52.4"/>
+    <xacro:property name="hip_torque_max" value="20.0"/>
     <xacro:property name="thigh_max" value="240"/>
     <xacro:property name="thigh_min" value="-60"/>
-    <xacro:property name="thigh_velocity_max" value="21"/>
-    <xacro:property name="thigh_torque_max" value="33.5"/>
+    <xacro:property name="thigh_velocity_max" value="28.6"/>
+    <xacro:property name="thigh_torque_max" value="55.0"/>
     <xacro:property name="calf_max" value="-52.5"/>
     <xacro:property name="calf_min" value="-154.5"/>
-    <xacro:property name="calf_velocity_max" value="21"/>
-    <xacro:property name="calf_torque_max" value="33.5"/>
+    <xacro:property name="calf_velocity_max" value="28.6"/>
+    <xacro:property name="calf_torque_max" value="55.0"/>
     <!-- dynamics inertial value -->
     <!-- trunk -->

File: robots/a1_description/xacro/gazebo.xacro (robot description, xacro)
@@ -9,5 +9,5 @@
     </gazebo>
     <!-- Show the trajectory of trunk center. -->
-    <gazebo>
+<!--     <gazebo>
         <plugin name="3dplot" filename="libLinkPlot3DPlugin.so">
             <frequency>10</frequency>
@@ -18,5 +18,5 @@
             </plot>
         </plugin>
-    </gazebo>
+    </gazebo> -->
     <!-- Show the trajectory of foot. You can add another trajectory about another foot. -->
     <!-- <gazebo>

File: robots/a1_description/xacro/robot.xacro (robot description, xacro)
@@ -8,6 +8,6 @@
     <!-- <xacro:include filename="$(find a1_gazebo)/launch/stairs.urdf.xacro"/> -->
     <!-- <xacro:stairs stairs="15" xpos="0" ypos="0" zpos="0" /> -->
-    <!-- Rollover Protection mode will add an additional stick on the top, use "true" or "false" to switch it. -->
-    <xacro:property name="rolloverProtection" value="false"/>
+    <!-- Rollover Protection mode will add an additional stick on the top, use 1 or 0 to switch it. -->
+    <xacro:property name="rolloverProtection" value= "0"/>
     <!-- Debug mode will hung up the robot, use "true" or "false" to switch it. -->
     <xacro:if value="$(arg DEBUG)">
@@ -55,5 +55,5 @@
         </inertial>
     </link>
-    <xacro:if value="${(rolloverProtection == 'true')}">
+    <xacro:if value="${rolloverProtection == 1}">
         <joint name="stick_joint" type="fixed">
             <parent link="trunk"/>
